Commit message: big changes

File: assets/urdf/fr3_crude.urdf (robot description, URDF)
Before this commit: robot fr3, 17 links, 16 joints
Links:
- removed link fr3_link0_sc
- removed link fr3_link1_sc
- removed link fr3_link2_sc
- removed link fr3_link3_sc
- removed link fr3_link4_sc
- removed link fr3_link5_sc
- removed link fr3_link6_sc
- removed link fr3_link7_sc
- added link fr3_hand, mass 0.73; collision box size=0.14 0.24 0.18; visual box size=0.16 0.24 0.18
- added link fr3_hand_tcp, mass 1e-5
- added link fr3_leftfinger, mass 0.015
- added link fr3_rightfinger, mass 0.015
- link fr3_link0: mass None -> 0.629769; geometry collision cylinder length=0.03 radius=0.09; collision sphere radius=0.09
- link fr3_link1: mass None -> 4.970684; geometry collision cylinder length=0.283 radius=0.09; collision sphere radius=0.09
- link fr3_link2: mass None -> 0.646926; geometry collision cylinder length=0.12 radius=0.09; collision sphere radius=0.09
- link fr3_link3: mass None -> 3.228604; geometry collision cylinder length=0.15 radius=0.09; collision sphere radius=0.09
- link fr3_link4: mass None -> 3.587895; geometry collision cylinder length=0.12 radius=0.09; collision sphere radius=0.09
- link fr3_link5: mass None -> 1.225946; geometry collision cylinder length=0.25 radius=0.055; collision cylinder length=0.28 radius=0.09
- link fr3_link6: mass None -> 1.666555; geometry collision cylinder length=0.20 radius=0.08; visual cylinder length=0.20 radius=0.08
- link fr3_link7: mass None -> 0.735522; geometry collision cylinder length=0.28 radius=0.07; visual cylinder length=0.28 radius=0.07
- link fr3_link8: mass None -> 1e-5
Joints:
- removed joint fr3_link0_sc_joint
- removed joint fr3_link1_sc_joint
- removed joint fr3_link2_sc_joint
- removed joint fr3_link3_sc_joint
- removed joint fr3_link4_sc_joint
- removed joint fr3_link5_sc_joint
- removed joint fr3_link6_sc_joint
- removed joint fr3_link7_sc_joint
- added joint fr3_finger_joint1: type prismatic, parent fr3_hand, child fr3_leftfinger, origin xyz=0 0 0.0584 rpy=0 0 0, axis 0 1 0, limit lower=0.0 upper=0.04 effort=100 velocity=0.2
- added joint fr3_finger_joint2: type prismatic, parent fr3_hand, child fr3_rightfinger, origin xyz=0 0 0.0584 rpy=0 0 0, axis 0 -1 0, limit lower=0.0 upper=0.04 effort=100 velocity=0.2, mimic joint=fr3_finger_joint1
- added joint fr3_hand_joint: type fixed, parent fr3_link8, child fr3_hand, origin xyz=0 0 0 rpy=0 0 -0.7853981633974483
- added joint fr3_hand_tcp_joint: type fixed, parent fr3_hand, child fr3_hand_tcp, origin xyz=0 0 0.1034 rpy=0 0 0
